Commit message: made changes

File: src/description/urdf/robot_base.xacro (robot description, xacro)
@@ -92,5 +92,5 @@
       <parent link="base_link"/>
       <child link="camera_link"/>
-      <origin xyz="0.15 0 2" rpy="0 0.7 0"/>
+      <origin xyz="0.15 0 2" rpy="0 0.4 0"/>
     </joint>
     <xacro:macro name="wheel" params="name x y">

Commit message: Swap turret and base camera roles, update naming, and fix RViz configuration

File: src/description/urdf/robot_base.xacro (robot description, xacro)
@@ -148,33 +148,33 @@
   <dynamics damping="0.1" friction="0.1"/>
 </joint>
-<!-- ================= CAMERA ================= -->
+<!-- ================= TURRET CAMERA ================= -->
+<link name="turret_camera_link">
+  <visual>
+    <geometry>
+      <box size="0.05 0.05 0.05"/>
+    </geometry>
+    <material name="Red">
+      <color rgba="1 0 0 1"/>
+    </material>
+  </visual>
+  <collision>
+    <geometry>
+      <box size="0.05 0.05 0.05"/>
+    </geometry>
+  </collision>
+  <inertial>
+    <mass value="0.3"/>
+    <origin xyz="0 0 0"/>
+    <inertia ixx="0.005" iyy="0.005" izz="0.005"
+             ixy="0" ixz="0" iyz="0"/>
+  </inertial>
+</link>
+<joint name="turret_camera_joint" type="fixed">
+  <parent link="tilt_link"/>
+  <child link="turret_camera_link"/>
+  <origin xyz="0 0 0.03"/>
+</joint>
+<!-- ================= LANE CAMERA ================= -->
 <link name="camera_link">
-  <visual>
-    <geometry>
-      <box size="0.05 0.05 0.05"/>
-    </geometry>
-    <material name="red">
-      <color rgba="1 0 0 1"/>
-    </material>
-  </visual>
-  <collision>
-    <geometry>
-      <box size="0.05 0.05 0.05"/>
-    </geometry>
-  </collision>
-  <inertial>
-    <mass value="0.3"/>
-    <origin xyz="0 0 0"/>
-    <inertia ixx="0.005" iyy="0.005" izz="0.005"
-             ixy="0" ixz="0" iyz="0"/>
-  </inertial>
-</link>
-<joint name="camera_joint" type="fixed">
-  <parent link="tilt_link"/>
-  <child link="camera_link"/>
-  <origin xyz="0 0 0.03"/>
-</joint>
-<!-- ================= SIDE CAMERA ================= -->
-<link name="side_camera_link">
   <visual>
     <geometry>
@@ -197,8 +197,8 @@
   </inertial>
 </link>
-<joint name="side_camera_joint" type="fixed">
+<joint name="camera_joint" type="fixed">
   <parent link="base_link"/>
-  <child link="side_camera_link"/>
-  <origin xyz="0.15 0 2" rpy="0 0.4 0"/>
+  <child link="camera_link"/>
+  <origin xyz="0.15 0 2" rpy="0 0.4 0"/> <!-- chcanged camera and turret positions-->
 </joint>
     <xacro:macro name="wheel" params="name x y">

File: src/description/urdf/robot_sensors.xacro (robot description, xacro)
@@ -41,8 +41,8 @@
     </gazebo>
     <gazebo reference="camera_link">
-      <sensor name="turret_camera_sensor" type="camera">
+      <sensor name="camera_sensor" type="camera">
         <always_on>true</always_on>
         <update_rate>30</update_rate>
-        <topic>/turret_camera/image_raw</topic>
+        <topic>/camera/image_raw</topic>
         <camera>
           <horizontal_fov>1.047</horizontal_fov>
@@ -59,9 +59,9 @@
       </sensor>
     </gazebo>
-    <gazebo reference="side_camera_link">
-  <sensor name="camera_sensor" type="camera">
+    <gazebo reference="turret_camera_link">
+  <sensor name="turret_camera_sensor" type="camera">
     <always_on>true</always_on>
     <update_rate>30</update_rate>
-    <topic>/camera/image_raw</topic>
+    <topic>/turret_camera/image_raw</topic>
     <camera>
       <horizontal_fov>1.047</horizontal_fov>
